File: ocs-tray-mezzanine-adapter-v1.kicad_pcb (KiCad board)
At the start: 4 copper layers, 53.3 x 44.3 mm, 43 parts, among them J1 SEAF-20-06.5-L-08-2-A-K-TR, J2 USB3_A, J3 45558-0003, J4 Conn_01x03, J5 Conn_01x03, SW1 SW_DIP_x02, SW2 SW_Push, U1 TSR_1-2433, U2 SI53154

Commit message: Revision A done
Parts:
- added REF***: OSHW-Logo2_7.3x6mm_SilkScreen, Symbols:OSHW-Logo2_7.3x6mm_SilkScreen, B.Cu at (201.2, 59.9)
Connections:
- net Net-(J1-PadB1) renamed /PCIE_RX_7_P
- net Net-(J1-PadB2) renamed /PCIE_RX_7_N
- net Net-(J1-PadD1) renamed /PCIE_RX_15_P
- net Net-(J1-PadD2) renamed /PCIE_RX_15_N
- net Net-(J1-PadF1) renamed /PCIE_TX_7_P
- net Net-(J1-PadF2) renamed /PCIE_TX_7_N
- net Net-(J1-PadH1) renamed /PCIE_TX_15_P
- net Net-(J1-PadH2) renamed /PCIE_TX_15_N
Routing:
- net /PCIE_TX_15_P: track 0.00 -> 3.15 mm, vias 0 -> 1
- net /PCIE_TX_15_N: track 0.00 -> 2.52 mm, vias 0 -> 1
- net GND: track 135.3 -> 133.8 mm, vias 78 -> 76
- net /PCIE_TX_7_N: track 0.00 -> 0.90 mm, vias 0 -> 1
- net /PCIE_RX_7_P: track 0.00 -> 0.90 mm, vias 0 -> 1
- net /PCIE_RX_15_N: track 0.00 -> 0.90 mm, vias 0 -> 1
- net /PCIE_TX_7_P: track 0.00 -> 0.90 mm, vias 0 -> 1
- net /PCIE_RX_7_N: track 0.00 -> 0.90 mm, vias 0 -> 1
- net /PCIE_RX_15_P: track 0.00 -> 0.90 mm, vias 0 -> 1
Other:
- board text added: "1"
- board text added: "2"
- board text added: "3"
- board text added: "4"
- board text added: "Licensed under CERN-OHL-P v2.0"
